Commit message: Refactor base_link to robot rotation center
Make base_link conform to ROS mobile robot conventions:
- X axis points to visual front (was visual rear in SolidWorks export)
- Y axis points to robot left, Z axis up
- Origin moved to wheel midpoint, so in-place rotation no longer
  makes base_link orbit a 0.5m circle
- laser_link now fully aligned with base_link (X to visual front)

Result:
- /cmd_vel linear.x > 0 moves robot toward visual front
- 2D Pose Estimate arrow direction matches visual front
- AMCL particle cloud and pose are oriented correctly

All changes are localized to tjark_agv.urdf:
- visual/collision origin: 180 deg yaw + translation to wheel midpoint
- body_to_base, 2 wheel and 4 caster joints: xyz and rpy adjusted
  to reflect frame flip + origin relocation
- laser_to_body: pitch sign flipped to compensate base_link rotation

No changes to controller/sensor xacro, launch files, world, maps,
SLAM/AMCL/move_base configs.

File: src/tjark_agv/urdf/tjark_agv.urdf (robot description, URDF)
Before this commit: robot tjark_agv, 10 links, 9 joints
Joints:
- joint LB_to_base: origin xyz=0.15553 -0.59031 -0.11632 rpy=-1.5708 0 1.5708 -> xyz=-0.138 0.094005 0.0055 rpy=-1.5708 0 -1.5708
- joint LF_to_base: origin xyz=-0.12047 -0.59031 -0.11632 rpy=-3.1416 0 -1.5708 -> xyz=0.138 0.094005 0.0055 rpy=-3.1416 0 1.5708
- joint RB_to_base: origin xyz=0.15553 -0.40231 -0.11632 rpy=3.1416 0 -1.5708 -> xyz=-0.138 -0.093995 0.0055 rpy=3.1416 0 1.5708
- joint RF_to_base: origin xyz=-0.12047 -0.40231 -0.11632 rpy=-3.1416 0 -1.5708 -> xyz=0.138 -0.093995 0.0055 rpy=-3.1416 0 1.5708
- joint body_to_base: origin xyz=0.0910304262953284 -0.439267303074538 0.0528804871592127 rpy=1.5707963267949 0 1.5707963267949 -> xyz=-0.0735004262953284 -0.057037696925462 0.1747004871592127 rpy=1.5707963267949 0 -1.5707963267949
- joint laser_to_body: origin xyz=-0.057039 -0.041697 -0.23945 rpy=-1.5708 -1.5708 0 -> xyz=-0.057039 -0.041697 -0.23945 rpy=-1.5708 1.5708 0
- joint left_to_base: origin xyz=0.01753 -0.68851 -0.12182 rpy=-1.5708 0 0 -> xyz=0 0.192205 0 rpy=-1.5708 0 3.14159265358979
- joint right_to_base: origin xyz=0.01753 -0.3041 -0.12182 rpy=-1.5708 0 0 -> xyz=0 -0.192205 0 rpy=-1.5708 0 3.14159265358979
