Commit message: Save SLAM mapping and localization progress before v2 model
This commit preserves the old-model (v1) stage achievements before
introducing the teacher's corrected tjark_agv model (v2).

Included:
- Old model URDF fixes (controller, sensor, base_link rotation center)
- Cartographer config tuning (tjark_agv_2d.lua)
- Cartographer localization launch and config
- AMCL localization launch and RViz config
- Gmapping tuned launch
- Square maze world and launch
- Camera wide xacro
- Direction verification RViz config

File: src/tjark_agv/urdf/tjark_agv.controller.xacro (robot description, xacro)
@@ -20,6 +20,6 @@
             <leftJoint>left_to_base</leftJoint>
             <rightJoint>right_to_base</rightJoint>
-            <wheelSeparation>0.38441</wheelSeparation>
-            <wheelDiameter>0.149</wheelDiameter>
+            <wheelSeparation>0.316</wheelSeparation>
+            <wheelDiameter>0.125</wheelDiameter>
             <broadcastTF>1</broadcastTF>
             <wheelTorque>30</wheelTorque>

File: src/tjark_agv/urdf/tjark_agv.sensor.xacro (robot description, xacro)
@@ -7,5 +7,5 @@
             <pose>0 0 0 0 0 0</pose>
             <visualize>$(arg laser_visual)</visualize>
-            <update_rate>7</update_rate>
+            <update_rate>60</update_rate>
             <ray>
                 <scan>
@@ -13,6 +13,6 @@
                     <samples>720</samples>
                     <resolution>0.5</resolution>
-                    <min_angle>0.0</min_angle>
-                    <max_angle>6.28319</max_angle>
+                    <min_angle>-1.5708</min_angle>
+                    <max_angle>1.5708</max_angle>
                     </horizontal>
                 </scan>
@@ -25,5 +25,5 @@
                     <type>gaussian</type>
                     <mean>0.0</mean>
-                    <stddev>0.01</stddev>
+                    <stddev>0.0</stddev>
                 </noise>
             </ray>

File: src/tjark_agv/urdf/tjark_agv.urdf (robot description, URDF)
Before this commit: robot tjark_agv, 10 links, 9 joints
Links:
- added link base_footprint
- link left_wheel: mass 0.223430950895449 -> 0.223430950718916
- link right_wheel: mass 0.223430950718916 -> 0.223430950895449
Joints:
- added joint base_footprint_to_base: type fixed, parent base_footprint, child base_link, origin xyz=0 0 0 rpy=0 0 0
